File: ESPFLASHER.kicad_pcb (KiCad board)
At the start: 2 copper layers, 40 x 21 mm, 23 parts, among them J1 USB_B_Micro, J2 PROG, Q1 S8050, Q2 S8050, Q3 2N7002, Q4 2N7002, U1 AMS1117-3.3, U2 SRV05-4, U3 CH340C

Commit message: Update V2 programmer with USB-C and simplified indicators
Replace the USB connector with a USB-C USB 2.0 receptacle and independent CC pull-downs. Remove RX/TX indicators and move the power LED beside J2. Include regulator, clearance, labeling, and USB routing improvements, with refreshed documentation and manufacturing outputs.

Validation: ERC and PCB DRC report zero errors; no unconnected pads or schematic parity issues. Library warnings remain documented. Hardware has not been tested.
Parts:
- removed D1: RX, LED_SMD:LED_0603_1608Metric
- removed D2: TX, LED_SMD:LED_0603_1608Metric
- removed Q3, Q4: 2N7002, Package_TO_SOT_SMD:SOT-23
- removed R3, R4, R5, R6: 1k, Resistor_SMD:R_0603_1608Metric
- added R8: 5.1k, Resistor_SMD:R_0603_1608Metric, F.Cu at (86.5, 43.5)
- added R9: 5.1k, Resistor_SMD:R_0603_1608Metric, F.Cu at (86.5, 56.2)
- J1: value USB_B_Micro -> TYPE-C-31-M-12; footprint Connector_USB:USB_Micro-B_Amphenol_10118194_Horizontal -> Connector_USB:USB_C_Receptacle_HRO_TYPE-C-31-M-12
- U1: value AMS1117-3.3 -> TLV1117LV33DCYR
- moved R7 11.0 mm to (107.5, 55.6), turned to 180 degrees
- moved D3 4.72 mm to (111.2, 55.6), turned to 180 degrees
- moved U2 1.49 mm to (90.5, 50.8)
- moved J1 0.43 mm to (83.2, 50.0)
Routing:
- net /PC_TXD: track 56.7 -> 45.3 mm
- net /PC_RXD: track 44.9 -> 35.3 mm, vias 4 -> 3
- net /CC1: track 0.00 -> 8.97 mm, vias 0 -> 2
- net Net-(D2-K): track 7.50 -> 0.00 mm, vias 2 -> 0
- net /CC2: track 0.00 -> 6.52 mm, vias 0 -> 2
- net +3V3: track 75.1 -> 68.9 mm, vias 9 -> 11
- net Net-(D1-K): track 5.94 -> 0.00 mm, vias 2 -> 0
- net VBUS: track 19.8 -> 24.6 mm
- net Net-(Q4-G): track 3.18 -> 0.00 mm
- net GND: track 33.0 -> 30.7 mm, vias 10 -> 12
- net Net-(Q3-G): track 2.21 -> 0.00 mm
- net Net-(D2-A): track 2.03 -> 0.00 mm
- net Net-(D1-A): track 2.02 -> 0.00 mm
- net /D-: track 18.0 -> 16.2 mm, vias 2 -> 3
Other:
- board text added: "3V3"
- board text added: "EN"
- board text added: "ESP8266/32 PROGRAMMER V2"
- board text added: "GND"
- board text added: "IO0"
- board text added: "PWR"
- board text added: "RX"
- board text added: "TX"
- board text removed: "ESP8266/32 PROGRAMMER v2"
- board text removed: "GND RX TX IO0 EN VCC"

Commit message: Mark USB-C board V3 and add connector 3D preview
Other:
- board text added: "ESP8266/32 PROGRAMMER V3"
- board text removed: "ESP8266/32 PROGRAMMER V2"
Changed lines of the file:
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@@
 	(paper "A4")
 	(title_block
-		(rev "2")
+		(rev "3")
 	)
 	(layers
@@
 		)
 		(embedded_fonts no)
-		(model "${KICAD9_3DMODEL_DIR}/Connector_USB.3dshapes/USB_C_Receptacle_HRO_TYPE-C-31-M-12.step"
+		(model "${KIPRJMOD}/3dmodels/HRO_TYPE-C-31-M-12.step"
 			(offset
-				(xyz 0 0 0)
+				(xyz -4.47 -3.65 0)
 			)
 			(scale
@@
 			)
 			(rotate
-				(xyz 0 0 0)
+				(xyz -90 0 0)
 			)
 		)
@@
 		)
 	)
-	(gr_text "ESP8266/32\nPROGRAMMER V2"
+	(gr_text "ESP8266/32\nPROGRAMMER V3"
 		(at 107.5 50.6 0)
 		(layer "F.SilkS")
