File: ESPFLASHER.kicad_sch (KiCad schematic)
At the start: 23 parts, among them J1 USB_B_Micro, J2 PROG, Q1 S8050, Q2 S8050, Q3 2N7002, Q4 2N7002, U1 AMS1117-3.3, U2 SRV05-4, U3 CH340C

Commit message: Remanufacturing, update to latest KiCAD
Signed-off-by: Denys Fedoryshchenko <denys.f@collabora.com>
Parts:
- C1, C2: JLCPCB (none) -> C2762594
- C3, C4: JLCPCB (none) -> C59302
- D1, D2, D3: JLCPCB (none) -> C2286
- J1: JLCPCB (none) -> C132563
- Q1, Q2: JLCPCB (none) -> C2150
- Q3, Q4: JLCPCB (none) -> C8545
- R1, R2: JLCPCB (none) -> C25804
- R3, R4, R5, R6, R7: JLCPCB (none) -> C21190
- U1: JLCPCB (none) -> C6186
- U2: JLCPCB (none) -> C558418
- U3: JLCPCB (none) -> C7464026

Commit message: Update V2 programmer with USB-C and simplified indicators
Replace the USB connector with a USB-C USB 2.0 receptacle and independent CC pull-downs. Remove RX/TX indicators and move the power LED beside J2. Include regulator, clearance, labeling, and USB routing improvements, with refreshed documentation and manufacturing outputs.

Validation: ERC and PCB DRC report zero errors; no unconnected pads or schematic parity issues. Library warnings remain documented. Hardware has not been tested.
Parts:
- removed D1: RX, LED_SMD:LED_0603_1608Metric, symbol Device:LED_Small
- removed D2: TX, LED_SMD:LED_0603_1608Metric, symbol Device:LED_Small
- removed Q3, Q4: 2N7002, Package_TO_SOT_SMD:SOT-23, symbol Transistor_FET:2N7002
- removed R3, R4, R5, R6: 1k, Resistor_SMD:R_0603_1608Metric, symbol Device:R_Small
- added R8, R9: 5.1k, Resistor_SMD:R_0603_1608Metric, symbol Device:R_Small
- J1: value USB_B_Micro -> TYPE-C-31-M-12; footprint Connector_USB:USB_Micro-B_Amphenol_10118194_Horizontal -> Connector_USB:USB_C_Receptacle_HRO_TYPE-C-31-M-12; symbol Connector:USB_B_Micro -> Connector:USB_C_Receptacle_USB2.0_16P; JLCPCB C132563 -> C165948
- U1: value AMS1117-3.3 -> TLV1117LV33DCYR; symbol Regulator_Linear:AMS1117-3.3 -> ESPFLASHER:TLV1117LV33DCYR; JLCPCB C6186 -> C15578
Connections:
- net D+: now also J1.A6 (D+), J1.B6 (D+); no longer J1.3 (D+)
- net D-: now also J1.A7 (D-), J1.B7 (D-); no longer J1.2 (D-)
- net GND: now also J1.A1 (GND), J1.A12 (GND), J1.B1 (GND), J1.B12 (GND), J1.S1 (SHIELD), R8.2, R9.2; no longer J1.5 (GND), J1.6 (Shield)
- net VBUS: now also J1.A4 (VBUS), J1.A9 (VBUS), J1.B4 (VBUS), J1.B9 (VBUS); no longer J1.1 (VBUS)
- new net CC1: J1.A5 (CC1), R8.1
- new net CC2: J1.B5 (CC2), R9.1
- no-connect marks 6 -> 7
Other:
- note added: "3.3V power indicator"
- note added: "Programming header"
- note added: "USB-C: USB 2.0, 5 V sink Separate 5.1k Rd on CC1 and CC2"
- note removed: "Connectors"
- note removed: "Errata: LED might need to be inverted, they are ON on idle."
- note removed: "Indicators (RX, TX, Power)"
